File: devboard.sch (EAGLE design)
At the start: 23 parts, among them Q1 CRYSTALX22, X1 MICROMATCH-8

Commit message: added eeprom for storing mac address and 2x13 pin connector
Parts:
- added JP1: (no value), pinhead:PINHD-2X13
- added R10, R9: 4k7, rcl:R-EU_R0603
- added R2, R4, R5, R6, R7, R8: 0R, rcl:R-EU_R0603
- added U2: 24LC32A/SN, hexabus:24LC32A/SN
Connections:
- new net N$10: R5.1, R8.2, U2.A2
- new net N$4: R2.1, R6.2, U2.A0
- new net N$9: R4.1, R7.2, U2.A1
- new net SCL: JP1.5, R10.1, U2.SCL
- new net SDA: JP1.3, R9.1, U2.SDA
- net AT_RST: now also JP1.16
- net GND: now also JP1.14, JP1.20, JP1.25, JP1.6, JP1.9, R6.1, R7.1, R8.1, U2.VSS, U2.WP
- net IRQ: now also JP1.15
- net MISO: now also JP1.21
- net MOSI: now also JP1.19
- net SCLK: now also JP1.23
- net SEL1: now also JP1.24
- net SLP_TR: now also JP1.18
- net VCC: now also JP1.1, R10.2, R2.2, R4.2, R5.2, R9.2, U2.VCC
Other:
- note added: "alternative"
- note added: "either populate pull up or pull down resistor to set I2C ID"
